File: Adem rev1/ADEM.kicad_pcb (KiCad board)
At the start: 2 copper layers, 95 x 46 mm, 28 parts, among them P1 CONN_buzz, P2 CONN_01X03, P3 CONN_01X04, Q1 NPN, U3 ESP8266_THING, U4 MPU6050, U5 NVSRAM, U6 BMP180, U7 HTU21D

Commit message: I2C-GPS initial design
Parts:
- added R4: R, Resistors_SMD:R_1206_HandSoldering, F.Cu at (183.7, 62.9)
- U4: footprint ADEM:MPU6050_angled -> ADEM:MPU6050_angled_down
- moved P-I2C-GPS1 20.0 mm to (204.6, 63.9)
- moved Q1 12.2 mm to (199.4, 55.4), turned to 180 degrees
- moved R3 9.16 mm to (199.5, 77.6)
- moved R2 9.06 mm to (199.5, 75.1)
- moved S2 7.85 mm to (194.2, 73.2), turned to 0 degrees
- moved C1 7.15 mm to (187.9, 57.0), turned to 180 degrees
- moved S1 6.59 mm to (196.8, 72.8), turned to 90 degrees
- moved C7 5.89 mm to (189.9, 52.3), turned to 180 degrees
- moved U4 5.34 mm to (179.7, 65.5)
- moved A_MPU 4.99 mm to (183.1, 73.2), turned to 270 degrees
- moved D1 4.82 mm to (197.0, 60.3), turned to 180 degrees
- moved R1 4.43 mm to (187.8, 59.8)
- moved C6 3.03 mm to (196.8, 63.8)
- moved C2 0.52 mm to (199.5, 80.1)
- moved C3 0.25 mm to (201.4, 69.8)
- renumbered GS_MPU1 to A_MPU, GS_NV1 to A_NV1, GS_NV2 to A_NV2, GS_NV3 to A_NV3, GS1 to S1, GS2 to S2
Routing:
- net VCC: track 95.9 -> 196.3 mm
- net INT: track 0.35 -> 76.9 mm
- net NEO_PXL: track 0.35 -> 60.5 mm
- net GND: track 16.9 -> 62.4 mm, vias 4 -> 10
- net SCL: track 48.0 -> 84.2 mm
- net BUZZ: track 0.35 -> 36.1 mm
- net (no net): track 83.4 -> 50.0 mm, vias 1 -> 0
- net SDA: track 55.9 -> 86.8 mm
- net Net-(D1-Pad2): track 1.43 -> 14.4 mm
- net Net-(Q1-Pad2): track 0.00 -> 8.88 mm
- net Net-(GS_MPU1-Pad2): track 0.00 -> 6.02 mm
- net Net-(GS2-Pad2): track 0.00 -> 5.65 mm
- net Net-(P3-Pad2): track 4.06 -> 9.45 mm
- net Net-(P3-Pad3): track 4.06 -> 9.45 mm
- net Net-(GS1-Pad1): track 0.08 -> 2.91 mm
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- added copper zone on F.Cu, net VCC
Other:
- board size 95 x 46 mm -> 71 x 46.2 mm
