File: Adem rev1/ADEM.sch (KiCad schematic (older format))
At the start: 28 parts, among them P1 CONN_buzz, P2 CONN_01X03, P3 CONN_01X04, Q1 NPN, U3 ESP8266_THING, U4 MPU6050, U5 NVSRAM, U6 BMP180, U7 HTU21D

Commit message: I2C-GPS initial design
Parts:
- added R4: R, Resistors_SMD:R_1206_HandSoldering, symbol R
- GS2: value GS2 -> S2
- U4: footprint ADEM:MPU6050_angled -> ADEM:MPU6050_angled_down
- renumbered P-I2C-GPS1 to P_I2CGPS1
Connections:
- net INT: now also R4.2
- net VCC: now also R4.1
Changed lines of the file:
@@
 F 0 "U4" H 9450 1600 60  0000 C CNN
 F 1 "MPU6050" H 9400 2500 60  0000 C CNN
-F 2 "ADEM:MPU6050_angled" H 9450 1600 60  0001 C CNN
+F 2 "ADEM:MPU6050_angled_down" H 9450 1600 60  0001 C CNN
 F 3 "~" H 9450 1600 60  0000 C CNN
 	1    9450 2100
@@
 U 1 1 5638ED57
 P 7200 1800
-F 0 "GS1" H 7300 1950 50  0000 C CNN
+F 0 "S1" H 7300 1950 50  0000 C CNN
 F 1 "GS1" H 7300 1651 40  0000 C CNN
 F 2 "Connect:GS2" V 7274 1800 30  0000 C CNN
@@
 U 1 1 5638EDB5
 P 8000 3950
-F 0 "GS_NV2" H 8050 4150 50  0000 C CNN
+F 0 "A_NV2" H 8050 4150 50  0000 C CNN
 F 1 "GS_A1" H 8050 3751 40  0000 C CNN
 F 2 "Connect:GS3" V 8088 3876 30  0000 C CNN
@@
 U 1 1 5638EEB5
 P 8000 4400
-F 0 "GS_NV3" H 8050 4600 50  0000 C CNN
+F 0 "A_NV3" H 8050 4600 50  0000 C CNN
 F 1 "GS_A2" H 8050 4201 40  0000 C CNN
 F 2 "Connect:GS3" V 8088 4326 30  0000 C CNN
@@
 U 1 1 5638EECA
 P 8000 3500
-F 0 "GS_NV1" H 8050 3700 50  0000 C CNN
+F 0 "A_NV1" H 8050 3700 50  0000 C CNN
 F 1 "GS_A0" H 8050 3301 40  0000 C CNN
 F 2 "Connect:GS3" V 8088 3426 30  0000 C CNN
@@
 U 1 1 5638F172
 P 7700 2750
-F 0 "GS_MPU1" H 7750 2950 50  0000 C CNN
+F 0 "A_MPU1" H 7750 2950 50  0000 C CNN
 F 1 "GS_A0" H 7750 2551 40  0000 C CNN
 F 2 "Connect:GS3" V 7788 2676 30  0000 C CNN
@@
 P 7550 1750
 F 0 "GS2" H 7650 1900 50  0000 C CNN
-F 1 "GS2" H 7650 1601 40  0000 C CNN
+F 1 "S2" H 7650 1601 40  0000 C CNN
 F 2 "Connect:GS2" V 7624 1750 30  0000 C CNN
 F 3 "" H 7550 1750 60  0000 C CNN
@@
 	7700 3600 7850 3600
 $Comp
-L CONN_01X05 P-I2C-GPS1
+L CONN_01X05 P_I2CGPS1
 U 1 1 57BA2962
 P 2700 2450
-F 0 "P_I2CGPS" H 2700 2750 50  0000 C CNN
+F 0 "P_I2CGPS1" H 2700 2750 50  0000 C CNN
 F 1 "CONN_01X05" V 2800 2450 50  0000 C CNN
 F 2 "Pin_Headers:Pin_Header_Angled_1x05" H 2700 2450 50  0001 C CNN
@@
 Wire Wire Line
 	2500 2450 1800 2450
+$Comp
+L R R4
+U 1 1 57BB4869
+P 1900 2050
+F 0 "R4" V 1980 2050 40  0000 C CNN
+F 1 "R" V 1907 2051 40  0000 C CNN
+F 2 "Resistors_SMD:R_1206_HandSoldering" V 1830 2050 30  0001 C CNN
+F 3 "~" H 1900 2050 30  0000 C CNN
+	1    1900 2050
+	1    0    0    -1
+$EndComp
+$Comp
+L VCC #PWR035
+U 1 1 57BB49AA
+P 1900 1800
+F 0 "#PWR035" H 1900 1900 30  0001 C CNN
+F 1 "VCC" H 1900 1900 30  0000 C CNN
+F 2 "" H 1900 1800 60  0000 C CNN
+F 3 "" H 1900 1800 60  0000 C CNN
+	1    1900 1800
+	1    0    0    -1
+$EndComp
+Wire Wire Line
+	1900 1800 1900 1900
+Wire Wire Line
+	1900 2200 1900 2550
+Connection ~ 1900 2550
 $EndSCHEMATC
